File: board/A2E_IOU_spkr/A2E_IOU_spkr.kicad_pcb (KiCad board)
At the start: 2 copper layers, 33 x 53.3 mm, 5 parts, among them J1 IOU_Socket, J2 PCB_Socket, J3 Test, U1 GAL16V8

Commit message: Update PCB
Connections:
- J1 pad 8: /SPKR -> (no net)
- U1 pad 1: /PHI0 -> Net-(U1-Pad1)
- U1 pad 12: Net-(U1-Pad12) -> Net-(U1-Pad1)
- U1 pad 13: Net-(U1-Pad13) -> (no net)
- U1 pad 14: Net-(U1-Pad14) -> (no net)
- U1 pad 15: Net-(U1-Pad15) -> (no net)
- U1 pad 16: Net-(U1-Pad16) -> (no net)
- U1 pad 17: Net-(U1-Pad17) -> (no net)
- U1 pad 18: Net-(U1-Pad18) -> (no net)
- U1 pad 7: GND -> /PHI0
Routing:
- net Net-(U1-Pad1): track 0.00 -> 23.5 mm
- net /PHI0: track 15.3 -> 9.51 mm
- net GND: track 92.2 -> 88.4 mm
